Commit message: updated packages to include scan message and proper transformations

File: puzzlebot_model/urdf/puzzlebot.urdf (robot description, URDF)
Before this commit: robot puzlebot, 4 links, 3 joints
Links:
- removed link base_footprint
- added link lidar_geom; visual cylinder length=0.05 radius=0.025
Joints:
- removed joint base_joint
- added joint base_to_lidar: type fixed, parent chasis, child lidar_geom, origin xyz=0 0 0.08  rpy=0 0 0
